Commit message: - added a draft ros2-control setup

File: description/robot.urdf.xacro (robot description, xacro)
@@ -3,4 +3,5 @@
     <xacro:include filename="robot_core.xacro" />
     <xacro:include filename="lidar.xacro" />
-    <xacro:include filename="gazebo_control.xacro"/>
+    <!-- <xacro:include filename="gazebo_control.xacro"/> -->
+    <xacro:include filename="ros2_control.xacro" />
 </robot>

File: description/robot_core.xacro (robot description, xacro)
@@ -49,5 +49,6 @@
         <collision>
             <geometry>
-                <cylinder radius="0.022" length="0.012"/>
+                <!-- <cylinder radius="0.022" length="0.012"/> -->
+                <sphere radius="0.022"/>
             </geometry>
         </collision>
@@ -75,5 +76,6 @@
         <collision>
             <geometry>
-                <cylinder radius="0.022" length="0.012"/>
+                <!-- <cylinder radius="0.022" length="0.012"/> -->
+                <sphere radius="0.022"/>
             </geometry>
         </collision>
